Commit message: Implement Python-like expression evaluation
Add ${...} expression syntax support for arithmetic, built-in functions,
and conditionals in xacro property values.

- New lexer for tokenizing ${expr}, $(extension), and $$ escapes
- Expression evaluator using pyisheval library
- Updated PropertyProcessor for recursive property evaluation
- Namespace handling (xacro: prefix or unprefixed only)

File: tests/data/property_test_multiple_expected.xacro (robot description, xacro)
@@ -1,4 +1,4 @@
 <?xml version="1.0"?>
 <robot name="test_robot" xmlns:xacro="http://www.ros.org/wiki/xacro">
- <box size="0.5 1.0 0.3"/>
+ <box size="0.5 1 0.3"/>
 </robot>
