Commit message: Address PR feedback on examples
Fix robot_with_args.xacro nested robot element (invalid URDF):
- Remove nested <robot> tag, use single root element
- Apply robot_name argument directly to root element

Fix advanced.rs to demonstrate configured features:
- Process robot_with_args.xacro instead of robot.xacro
- Now actually uses the passed arguments (robot_name)

Fix markdown lint issues (MD022):
- Add blank lines after all ### headings in README.md

File: examples/robot_with_args.xacro (robot description, xacro)
@@ -1,41 +1,37 @@
 <?xml version="1.0"?>
-<robot xmlns:xacro="http://www.ros.org/wiki/xacro">
+<robot xmlns:xacro="http://www.ros.org/wiki/xacro" name="$(arg robot_name)">
   <!-- Arguments that can be set from command line or API -->
   <xacro:arg name="robot_name" default="default_robot"/>
   <xacro:arg name="wheel_radius" default="0.1"/>
   <xacro:arg name="debug_mode" default="false"/>
-  <!-- Set the robot name from argument -->
-  <xacro:property name="name" value="$(arg robot_name)"/>
-  <robot name="${name}">
-    <!-- Conditional debug output -->
-    <xacro:if value="$(arg debug_mode)">
-      <link name="debug_marker">
-        <visual>
-          <geometry>
-            <sphere radius="0.01"/>
-          </geometry>
-        </visual>
-      </link>
-    </xacro:if>
-    <!-- Base link -->
-    <link name="base_link">
+  <!-- Conditional debug output -->
+  <xacro:if value="$(arg debug_mode)">
+    <link name="debug_marker">
       <visual>
         <geometry>
-          <box size="0.3 0.3 0.1"/>
+          <sphere radius="0.01"/>
         </geometry>
       </visual>
     </link>
-    <!-- Wheels using the radius argument -->
-    <xacro:macro name="wheel" params="side">
-      <link name="${side}_wheel">
-        <visual>
-          <geometry>
-            <cylinder radius="$(arg wheel_radius)" length="0.05"/>
-          </geometry>
-        </visual>
-      </link>
-    </xacro:macro>
-    <xacro:wheel side="left"/>
-    <xacro:wheel side="right"/>
-  </robot>
+  </xacro:if>
+  <!-- Base link -->
+  <link name="base_link">
+    <visual>
+      <geometry>
+        <box size="0.3 0.3 0.1"/>
+      </geometry>
+    </visual>
+  </link>
+  <!-- Wheels using the radius argument -->
+  <xacro:macro name="wheel" params="side">
+    <link name="${side}_wheel">
+      <visual>
+        <geometry>
+          <cylinder radius="$(arg wheel_radius)" length="0.05"/>
+        </geometry>
+      </visual>
+    </link>
+  </xacro:macro>
+  <xacro:wheel side="left"/>
+  <xacro:wheel side="right"/>
 </robot>
